Commit message: issue fixed

File: src/roverrobotics_description/urdf/rover_2wd.urdf (robot description, URDF)
Before this commit: robot rover_2wd, 8 links, 7 joints
Joints:
- joint base_to_chassis: origin xyz=0 0 0.125 -> xyz=-${wheel_x_offset} 0 0.125

Commit message: update

File: src/roverrobotics_description/urdf/rover_2wd.urdf (robot description, URDF)
Before this commit: robot rover_2wd, 8 links, 7 joints
Joints:
- joint fl_wheel_to_chassis: type continuous -> fixed
- joint fr_wheel_to_chassis: type continuous -> fixed
- joint rl_castor_to_chassis: type continuous -> fixed
- joint rl_ch_to_chassis: type continuous -> fixed
- joint rr_castor_to_chassis: type continuous -> fixed
- joint rr_ch_to_chassis: type continuous -> fixed
