Commit message: updated

File: src/roverrobotics_description/urdf/accessories/camera.urdf (robot description, URDF)
Before this commit: robot camera, 1 links, 1 joints
Links:
- removed link camera_link
- added link realsense_link
Joints:
- removed joint camera_to_payload
- added joint realsense_to_payload: type fixed, parent payload_link, child realsense_link, origin xyz=0 0 0.2 rpy=1.57 -1.57 0
